File: dcs_schematic_v3/dcs_schematic_v3.kicad_sch (KiCad schematic)
At the start: 56 parts, among them J1 691137710002, J2 1728307, Q1 IRLZ44N, U1 TLE2426CDR, U2 LM311DR, U3 LM2917N/NOPB, U4 HEF4030BT

Commit message: changed diode and updated datasheets/models accordingly. started PCB layout
Parts:
- removed D1: 1N5819G, 1N5819G:DIOAD1036W78L470D235, symbol Capstone_Diode:1N5819G
- added NT1, NT2: NetTie_2, NetTie:NetTie-2_SMD_Pad2.0mm, symbol Device:NetTie_2
- added U5: CDBW140-G, CapstoneLibrary:CDBW_Diode, symbol Capstone_DiodeActual:CDBW140-G
- Integrator1: renamed from Integrator; footprint OPA2197ID:SOIC127P599X175-8N -> CapstoneLibrary:OPA2197ID
- J1: footprint 691137710002:691137710002 -> CapstoneLibrary:TerminalBlock
- PWM_Gen1: renamed from PWM_Gen; footprint OPA2197ID:SOIC127P599X175-8N -> CapstoneLibrary:OPA2197ID
- Proportional/Control1: renamed from Proportional/Control; footprint OPA2197ID:SOIC127P599X175-8N -> CapstoneLibrary:OPA2197ID
- Setpoint/Error1: renamed from Setpoint/Error; footprint OPA2197ID:SOIC127P599X175-8N -> CapstoneLibrary:OPA2197ID
- U1: footprint TLE2426CDR:SOIC127P599X175-8N -> CapstoneLibrary:VREF_TLE2426CDR
- U2: footprint LM311DR:SOIC127P599X175-8N -> CapstoneLibrary:LM311DR
- U3: footprint M14A_TEX -> CapstoneLibrary:LM2917M
- U4: footprint SOT108-1_NXP -> CapstoneLibrary:XOR4030B
- to_motor1: renamed from to_motor; footprint 691137710002:691137710002 -> CapstoneLibrary:TerminalBlock
- renumbered C2_M+ to C2_M+1, C_Encoder to C_Encoder1, C_FV to C_FV1, C_FV_OUT to C_FV_OUT1, C_I to C_I1, C_M+ to C_M+1, C_Tri to C_Tri1, ENC_A_C to ENC_A_C1, ENC_A_R to ENC_A_R1, ENC_B_C to ENC_B_C1, ENC_B_R to ENC_B_R1, RA to RA1, RB to RB1, RC to RC1, RD to RD1, R_A_PU to R_A_PU1, R_BLEED to R_BLEED1, R_B_PU to R_B_PU1, R_ENC_OUT to R_ENC_OUT1, R_FP to R_FP1, R_FS to R_FS1, R_FV_OUT to R_FV_OUT1, R_Freq to R_Freq1, R_G to R_G1, R_GS to R_GS1, R_I to R_I1, R_P to R_P1, R_PU to R_PU1, R_SI to R_SI1, R_SP to R_SP1, SP_Cntl to SP_Cntl1
Connections:
- net +12V: now also NT1.2, NT2.2; no longer to_motor1.1
- net M-: now also U5.2
- net V_CONTROL: no longer Proportional/Control1.1 (OUTA), R_FP1.2, R_SP1.2
- new net M+: NT1.1, NT2.1, U5.1, to_motor1.1
- new net V_P: Proportional/Control1.1 (OUTA), R_FP1.2, R_SP1.2
- no-connect marks 8 -> 17

Commit message: progress on PCB layout
Parts:
- removed NT2: NetTie_2, NetTie:NetTie-2_SMD_Pad2.0mm, symbol Device:NetTie_2
Connections:
- net +12V: no longer C2_M+1.2, C_M+1.1
- net M+: now also C2_M+1.2, C_M+1.1
Other:
- moved on the sheet: NT1
Changed lines of the file:
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@@
 	)
 	(junction
-		(at 383.54 69.85)
+		(at 72.39 49.53)
 		(diameter 0)
 		(color 0 0 0 0)
 	)
 	(junction
-		(at 72.39 49.53)
+		(at 383.54 64.77)
 		(diameter 0)
 		(color 0 0 0 0)
@@
 	)
 	(junction
-		(at 383.54 64.77)
-		(diameter 0)
-		(color 0 0 0 0)
-	)
-	(junction
 		(at 78.74 49.53)
 		(diameter 0)
@@
 	)
 	(junction
-		(at 374.65 64.77)
-		(diameter 0)
-		(color 0 0 0 0)
-	)
-	(junction
 		(at 212.09 77.47)
 		(diameter 0)
@@
 	)
 	(junction
-		(at 388.62 64.77)
+		(at 77.47 176.53)
 		(diameter 0)
 		(color 0 0 0 0)
 	)
 	(junction
-		(at 77.47 176.53)
+		(at 374.65 64.77)
 		(diameter 0)
 		(color 0 0 0 0)
@@
 	(wire
 		(pts
-			(xy 363.22 64.77) (xy 374.65 64.77)
-		)
-		(stroke
-			(width 0)
-			(type default)
-		)
-	)
-	(wire
-		(pts
 			(xy 177.8 63.5) (xy 182.88 63.5)
 		)
@@
 	(wire
 		(pts
-			(xy 367.03 114.3) (xy 370.84 114.3)
+			(xy 383.54 67.31) (xy 383.54 64.77)
 		)
 		(stroke
@@
 	(wire
 		(pts
-			(xy 379.73 63.5) (xy 379.73 64.77)
+			(xy 367.03 114.3) (xy 370.84 114.3)
 		)
 		(stroke
@@
 	(wire
 		(pts
-			(xy 377.19 74.93) (xy 384.81 74.93)
+			(xy 379.73 63.5) (xy 379.73 64.77)
 		)
 		(stroke
@@
 	(wire
 		(pts
-			(xy 378.46 69.85) (xy 383.54 69.85)
+			(xy 377.19 74.93) (xy 384.81 74.93)
 		)
 		(stroke
@@
 	(wire
 		(pts
-			(xy 386.08 66.04) (xy 388.62 66.04)
-		)
-		(stroke
-			(width 0)
-			(type default)
-		)
-	)
-	(wire
-		(pts
 			(xy 80.01 173.99) (xy 80.01 176.53)
 		)
@@
 	(wire
 		(pts
+			(xy 383.54 64.77) (xy 389.89 64.77)
+		)
+		(stroke
+			(width 0)
+			(type default)
+		)
+	)
+	(wire
+		(pts
 			(xy 80.01 166.37) (xy 76.2 166.37)
 		)
@@
 	(wire
 		(pts
+			(xy 368.3 64.77) (xy 374.65 64.77)
+		)
+		(stroke
+			(width 0)
+			(type default)
+		)
+	)
+	(wire
+		(pts
 			(xy 182.88 54.61) (xy 187.96 54.61)
 		)
@@
 	(wire
 		(pts
-			(xy 388.62 66.04) (xy 388.62 64.77)
-		)
-		(stroke
-			(width 0)
-			(type default)
-		)
-	)
-	(wire
-		(pts
 			(xy 212.09 120.65) (xy 260.35 120.65)
 		)
@@
 	(wire
 		(pts
-			(xy 388.62 64.77) (xy 389.89 64.77)
-		)
-		(stroke
-			(width 0)
-			(type default)
-		)
-	)
-	(wire
-		(pts
 			(xy 134.62 77.47) (xy 144.78 77.47)
 		)
@@
 	(wire
 		(pts
-			(xy 386.08 69.85) (xy 386.08 66.04)
-		)
-		(stroke
-			(width 0)
-			(type default)
-		)
-	)
-	(wire
-		(pts
 			(xy 251.46 124.46) (xy 256.54 124.46)
 		)
@@
 	(wire
 		(pts
-			(xy 383.54 69.85) (xy 386.08 69.85)
-		)
-		(stroke
-			(width 0)
-			(type default)
-		)
-	)
-	(wire
-		(pts
 			(xy 184.15 90.17) (xy 184.15 91.44)
 		)
@@
 	(wire
 		(pts
-			(xy 377.19 67.31) (xy 378.46 67.31)
+			(xy 377.19 67.31) (xy 383.54 67.31)
 		)
 		(stroke
@@
 	(wire
 		(pts
-			(xy 378.46 69.85) (xy 378.46 67.31)
-		)
-		(stroke
-			(width 0)
-			(type default)
-		)
-	)
-	(wire
-		(pts
 			(xy 214.63 123.19) (xy 214.63 125.73)
 		)
@@
 		)
 	)
-	(label "M+"
-		(at 379.73 69.85 0)
+	(label "V_I"
+		(at 260.35 140.97 0)
 		(effects
 			(font
@@
 		)
 	)
-	(label "V_I"
-		(at 260.35 140.97 0)
+	(label "PWM"
+		(at 369.57 97.79 0)
 		(effects
 			(font
@@
 		)
 	)
-	(label "PWM"
-		(at 369.57 97.79 0)
+	(label "M+"
+		(at 377.19 64.77 0)
 		(effects
 			(font
@@
 	(symbol
 		(lib_id "Device:NetTie_2")
-		(at 383.54 67.31 90)
+		(at 365.76 64.77 180)
 		(unit 1)
 		(exclude_from_sim no)
@@
 		(dnp no)
 		(property "Reference" "NT1"
-			(at 381.508 71.12 90)
+			(at 371.602 63.246 0)
 			(effects
 				(font
 					(size 1.27 1.27)
 				)
-				(justify right)
+				(justify left)
 			)
 		)
 		(property "Value" "NetTie_2"
-			(at 381.508 73.66 90)
+			(at 371.602 60.706 0)
 			(effects
 				(font
 					(size 1.27 1.27)
 				)
-				(justify right)
+				(justify left)
 			)
 		)
 		(property "Footprint" "NetTie:NetTie-2_SMD_Pad2.0mm"
-			(at 383.54 67.31 0)
+			(at 365.76 64.77 0)
 			(effects
 				(font
@@
 		)
 		(property "Datasheet" "~"
-			(at 383.54 67.31 0)
+			(at 365.76 64.77 0)
 			(effects
 				(font
@@
 		)
 		(property "Description" "Net tie, 2 pins"
-			(at 383.54 67.31 0)
+			(at 365.76 64.77 0)
 			(effects
 				(font
@@
 		)
 		(instances
-			(project ""
+			(project "dcs_schematic_v3"
 				(path "/0fb55938-2350-4e3e-b10f-4d06caaaacd8"
 					(reference "NT1")
@@
 					(unit 1)
 				)
-			)
-		)
-	)
-	(symbol
-		(lib_id "Device:NetTie_2")
-		(at 386.08 64.77 180)
-		(unit 1)
-		(exclude_from_sim no)
-		(in_bom no)
-		(on_board yes)
-		(dnp no)
-		(property "Reference" "NT2"
-			(at 390.652 61.468 0)
-			(effects
-				(font
-					(size 1.27 1.27)
-				)
-				(justify right)
-			)
-		)
-		(property "Value" "NetTie_2"
-			(at 389.636 63.246 0)
-			(effects
-				(font
-					(size 1.27 1.27)
-				)
-				(justify right)
-			)
-		)
-		(property "Footprint" "NetTie:NetTie-2_SMD_Pad2.0mm"
-			(at 386.08 64.77 0)
-			(effects
-				(font
-					(size 1.27 1.27)
-				)
-				(hide yes)
-			)
-		)
-		(property "Datasheet" "~"
-			(at 386.08 64.77 0)
-			(effects
-				(font
-					(size 1.27 1.27)
-				)
-				(hide yes)
-			)
-		)
-		(property "Description" "Net tie, 2 pins"
-			(at 386.08 64.77 0)
-			(effects
-				(font
-					(size 1.27 1.27)
-				)
-				(hide yes)
-			)
-		)
-		(pin "1"
-		)
-		(pin "2"
-		)
-		(instances
-			(project "dcs_schematic_v3"
-				(path "/0fb55938-2350-4e3e-b10f-4d06caaaacd8"
-					(reference "NT2")
-					(unit 1)
-				)

Commit message: 80-90% done with first PCB layout. Need to rework parts to fix traces
Parts:
- added C_BP8: 0.1uF, Capacitor_SMD:C_0603_1608Metric_Pad1.08x0.95mm_HandSolder, symbol Device:C
- added R_VR1, R_VR2, R_VR3, R_VR4: 100, Resistor_SMD:R_0603_1608Metric_Pad0.98x0.95mm_HandSolder, symbol Device:R_US
- renumbered C_Bypass_1 to C_BP1, C_Bypass_2 to C_BP2, C_Bypass_3 to C_BP3, C_Bypass_4 to C_BP4, C_Bypass_5 to C_BP5, C_Bypass_6 to C_BP6, C_Bypass_7 to C_BP7, C_Encoder1 to C_Enc1, R_ENC_OUT1 to R_ENCOUT1
Connections:
- net +12V: now also C_BP8.2
- net GND: now also C_BP8.1
- net V_P: now also R_SP1.1; no longer R_SP1.2
- net V_REF: now also R_VR1.1, R_VR1.2, R_VR2.1, R_VR2.2, R_VR3.1, R_VR3.2, R_VR4.1, R_VR4.2
- net at Proportional/Control1.6 (-INB), R_FS1.1, R_SI1.1: now also R_SP1.2; no longer R_SP1.1
Other:
- moved on the sheet: R_SP1

Commit message: changed diode again. updated datasheets, models, etc.
Parts:
- removed U5: CDBW140-G, CapstoneLibrary:CDBW_Diode, symbol Capstone_DiodeActual:CDBW140-G
- added CR1: SK34A-LTP, CapstoneLibrary:SK32A-LTP_Diode, symbol Capstone_DiodeForReal:SK34A-LTP
Connections:
- net M+: now also CR1.1
- net M-: now also CR1.2
Changed lines of the file:
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@@
+	)
+	(symbol
+		(lib_id "Capstone_DiodeForReal:SK34A-LTP")
+		(at 389.89 74.93 90)
+		(unit 1)
+		(exclude_from_sim no)
+		(in_bom yes)
+		(on_board yes)
+		(dnp no)
+		(fields_autoplaced yes)
+		(property "Reference" "CR1"
+			(at 393.7 68.5799 90)
+			(effects
+				(font
+					(size 1.524 1.524)
+				)
+				(justify right)
+			)
+		)
+		(property "Value" "SK34A-LTP"
+			(at 393.7 71.1199 90)
+			(effects
+				(font
+					(size 1.524 1.524)
+				)
+				(justify right)
+			)
+		)
+		(property "Footprint" "CapstoneLibrary:SK32A-LTP_Diode"
+			(at 389.89 74.93 0)
+			(effects
+				(font
+					(size 1.27 1.27)
+					(italic yes)
+				)
+				(hide yes)
+			)
+		)
+		(property "Datasheet" "SK34A-LTP"
+			(at 389.89 74.93 0)
+			(effects
+				(font
+					(size 1.27 1.27)
+					(italic yes)
+				)
+				(hide yes)
+			)
+		)
+		(property "Description" ""
+			(at 389.89 74.93 0)
+			(effects
+				(font
+					(size 1.27 1.27)
+				)
+				(hide yes)
+			)
+		)
+		(pin "2"
+		)
+		(pin "1"
+		)
+		(instances
+			(project ""
+				(path "/0fb55938-2350-4e3e-b10f-4d06caaaacd8"
+					(reference "CR1")
+					(unit 1)
+				)
+			)
+		)
 	)
 	(symbol
@@
 					(unit 1)
 				)
-			)
-		)
-	)
-	(symbol
-		(lib_id "Capstone_DiodeActual:CDBW140-G")
-		(at 389.89 64.77 270)
-		(unit 1)
-		(exclude_from_sim no)
-		(in_bom yes)
-		(on_board yes)
-		(dnp no)
-		(fields_autoplaced yes)
-		(property "Reference" "U5"
-			(at 393.7 68.5799 90)
-			(effects
-				(font
-					(size 1.524 1.524)
-				)
-				(justify left)
-			)
-		)
-		(property "Value" "CDBW140-G"
-			(at 393.7 71.1199 90)
-			(effects
-				(font
-					(size 1.524 1.524)
-				)
-				(justify left)
-			)
-		)
-		(property "Footprint" "CapstoneLibrary:CDBW_Diode"
-			(at 389.89 64.77 0)
-			(effects
-				(font
-					(size 1.27 1.27)
-					(italic yes)
-				)
-				(hide yes)
-			)
-		)
-		(property "Datasheet" "CDBW140-G"
-			(at 389.89 64.77 0)
-			(effects
-				(font
-					(size 1.27 1.27)
-					(italic yes)
-				)
-				(hide yes)
-			)
-		)
-		(property "Description" ""
-			(at 389.89 64.77 0)
-			(effects
-				(font
-					(size 1.27 1.27)
-				)
-				(hide yes)
-			)
-		)
-		(pin "1"
-		)
-		(pin "2"
-		)
-		(instances
-			(project ""
-				(path "/0fb55938-2350-4e3e-b10f-4d06caaaacd8"
-					(reference "U5")
-					(unit 1)
-				)
