File: dcs_schematic_v3/dcs_schematic_v3.kicad_pcb (KiCad board)
At the start: 4 copper layers, 100 x 100 mm, 62 parts, among them J1 691137710002, J2 1728307, Q1 IRLZ44N, U1 TLE2426CDR, U2 LM311DR, U3 LM2917N/NOPB, U4 HEF4030BT, U5 CDBW140-G

Commit message: progress on PCB layout
Parts:
- removed NT2: NetTie_2, NetTie:NetTie-2_SMD_Pad2.0mm
- added REF**: TestPoint_Pad_D1.0mm, TestPoint:TestPoint_Pad_D1.0mm, F.Cu at (153.6, 87.0)
- added REF**: TestPoint_Pad_D1.0mm, TestPoint:TestPoint_Pad_D1.0mm, F.Cu at (156.7, 90.4)
- moved Setpoint/Error1 123.5 mm to (83.8, 98.2)
- moved Proportional/Control1 100.1 mm to (106.8, 98.5)
- moved R_H1 92.6 mm to (149.5, 121.4)
- moved Integrator1 84.0 mm to (123.5, 103.3)
- moved R_PU1 81.7 mm to (153.4, 95.7), turned to 180 degrees
- moved R_GS1 75.5 mm to (159.7, 87.0), turned to 180 degrees
- moved R_G1 73.2 mm to (155.4, 87.9), turned to -90 degrees
- moved R_Freq1 71.9 mm to (156.4, 122.5)
- moved U2 55.8 mm to (156.0, 100.2), turned to 90 degrees
- moved C_Tri1 55.6 mm to (167.7, 107.5)
- moved J2 47.1 mm to (186.8, 121.1)
- moved U3 40.4 mm to (201.0, 139.0)
- moved PWM_Gen1 39.4 mm to (157.3, 113.4), turned to 90 degrees
- moved R_B_PU1 20.6 mm to (250.2, 79.3)
- moved SP_Cntl1 18.4 mm to (99.4, 68.0)
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Connections:
- C2_M+1 pad 2: +12V -> /M+
- C_M+1 pad 1: +12V -> /M+
Routing:
- net /PWM: track 0.00 -> 11.4 mm
- net /M-: track 0.00 -> 10.7 mm
- net /V_TRI: track 0.00 -> 8.26 mm
- net Net-(Q1-G): track 0.00 -> 7.42 mm
- net /M+: track 0.00 -> 5.78 mm
- net GND: track 0.00 -> 2.33 mm, vias 0 -> 6
- net (no net): vias 2 -> 0
- added copper zone on In2.Cu, net +12V
- added copper zone on F.Cu, net /M+
- added copper zone on B.Cu, net GND
- added copper zone on In1.Cu, net GND
Other:
- board size 100 x 100 mm -> 72.5 x 100 mm

Commit message: 80-90% done with first PCB layout. Need to rework parts to fix traces
Parts:
- removed C_Bypass_1, C_Bypass_2, C_Bypass_3, C_Bypass_4, C_Bypass_5, C_Bypass_6, C_Bypass_7, C_Encoder1: 0.1uF, Capacitor_SMD:C_0603_1608Metric_Pad1.08x0.95mm_HandSolder
- removed the REF** at (158.2, 56.8)
- removed the REF** at (158.2, 135.0)
- removed the REF** at (99.3, 135.0)
- removed the REF** at (99.2, 57.0)
- added C_BP1: 0.1uF, Capacitor_SMD:C_0603_1608Metric_Pad1.08x0.95mm_HandSolder, F.Cu at (139.6, 93.0)
- added C_BP2: 0.1uF, Capacitor_SMD:C_0603_1608Metric_Pad1.08x0.95mm_HandSolder, F.Cu at (150.4, 102.1)
- added C_BP3: 0.1uF, Capacitor_SMD:C_0603_1608Metric_Pad1.08x0.95mm_HandSolder, F.Cu at (150.3, 110.1)
- added C_BP4: 0.1uF, Capacitor_SMD:C_0603_1608Metric_Pad1.08x0.95mm_HandSolder, F.Cu at (154.8, 110.8)
- added C_BP5: 0.1uF, Capacitor_SMD:C_0603_1608Metric_Pad1.08x0.95mm_HandSolder, F.Cu at (154.9, 100.6)
- added C_BP6: 0.1uF, Capacitor_SMD:C_0603_1608Metric_Pad1.08x0.95mm_HandSolder, F.Cu at (140.8, 70.9)
- added C_BP7: 0.1uF, Capacitor_SMD:C_0603_1608Metric_Pad1.08x0.95mm_HandSolder, F.Cu at (140.8, 88.3)
- added C_BP8: 0.1uF, Capacitor_SMD:C_0603_1608Metric_Pad1.08x0.95mm_HandSolder, F.Cu at (130.6, 104.7)
- added C_Enc1: 0.1uF, Capacitor_SMD:C_0603_1608Metric_Pad1.08x0.95mm_HandSolder, F.Cu at (126.8, 82.7)
- added REF**: TestPoint_Pad_D1.0mm, TestPoint:TestPoint_Pad_D1.0mm, F.Cu at (122.5, 69.9)
- added REF**: TestPoint_Pad_D1.0mm, TestPoint:TestPoint_Pad_D1.0mm, F.Cu at (117.7, 69.9)
- added REF**: TestPoint_Pad_D1.0mm, TestPoint:TestPoint_Pad_D1.0mm, F.Cu at (134.4, 102.6)
- added REF**: TestPoint_Pad_D1.0mm, TestPoint:TestPoint_Pad_D1.0mm, F.Cu at (120.1, 68.0)
- added R_VR1: 100, Resistor_SMD:R_0603_1608Metric_Pad0.98x0.95mm_HandSolder, F.Cu at (138.7, 102.5)
- added R_VR2: 100, Resistor_SMD:R_0603_1608Metric_Pad0.98x0.95mm_HandSolder, F.Cu at (138.7, 104.0)
- added R_VR3: 100, Resistor_SMD:R_0603_1608Metric_Pad0.98x0.95mm_HandSolder, F.Cu at (138.6, 105.5)
- added R_VR4: 100, Resistor_SMD:R_0603_1608Metric_Pad0.98x0.95mm_HandSolder, F.Cu at (136.2, 108.2)
- moved R_B_PU1 133.1 mm to (117.7, 66.8), turned to 90 degrees
- moved U4 123.2 mm to (135.8, 75.6)
- moved R_A_PU1 108.4 mm to (122.5, 66.8), turned to 90 degrees
- moved R_FV_OUT1 105.7 mm to (129.3, 86.8), turned to 90 degrees
- moved J1 102.8 mm to (159.0, 62.0), turned to 0 degrees
- moved R_BLEED1 101.1 mm to (139.2, 109.4), turned to -90 degrees
- moved R_ENCOUT 100.2 mm to (130.8, 82.0), turned to 90 degrees
- moved R_P1 99.6 mm to (143.5, 96.0), turned to -90 degrees
- moved ENC_B_R1 99.1 mm to (127.7, 76.9), turned to 180 degrees
- moved ENC_B_C1 98.8 mm to (127.7, 75.5)
- moved RA1 98.5 mm to (127.9, 91.2), turned to -90 degrees
- moved ENC_A_R1 97.2 mm to (127.7, 73.1), turned to 180 degrees
- moved ENC_A_C1 96.8 mm to (127.6, 71.6)
- moved C_FV1 92.2 mm to (129.9, 84.3), turned to 180 degrees
- moved C_FV_OUT1 91.3 mm to (130.8, 86.8), turned to -90 degrees
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- renumbered Integrator1 to Integrator, Proportional/Control1 to Proportional/Control, R_ENC_OUT1 to R_ENCOUT, U1 to VREF
Routing:
- net /V_REF: track 0.00 -> 91.3 mm
- net GND: track 2.33 -> 78.3 mm, vias 6 -> 48
- net +12V: track 0.00 -> 55.4 mm, vias 0 -> 16
- net /ENC_B: track 0.00 -> 19.5 mm
- net Net-(Setpoint/Error1--INB): track 0.00 -> 16.7 mm
- net /V_SET: track 0.00 -> 16.2 mm
- net /V_CONTROL: track 0.00 -> 16.2 mm
- net /ENC_A: track 0.00 -> 15.6 mm
- net /M+: track 5.78 -> 19.9 mm
- net Net-(Proportional/Control1--INA): track 0.00 -> 9.32 mm
- net Net-(Proportional/Control1--INB): track 0.00 -> 9.30 mm
- net Net-(PWM_Gen1--INB): track 0.00 -> 9.18 mm
- net /V_FEEDBACK: track 0.00 -> 8.85 mm
- net /V_SET_BUF: track 0.00 -> 8.73 mm
- net /ENC_OUT: track 0.00 -> 8.11 mm
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- removed copper zone on F.Cu, net /M+
Other:
- board outline removed
- board text added: "${REFERENCE}"
- board text added: "+12V"
- board text added: "ENC_A TEST"
- board text added: "ENC_B TEST"
- board text added: "VREF TEST"

Commit message: changed diode again. updated datasheets, models, etc.
Parts:
- removed U5: CDBW140-G, CapstoneLibrary:CDBW_Diode
- added CR1: SK34A-LTP, CapstoneLibrary:SK32A-LTP_Diode, F.Cu at (154.9, 81.5)
- moved NT1 1.85 mm to (150.8, 81.1)
- moved J1 1.40 mm to (159.0, 60.6)
- moved PS_DC1 1.40 mm to (150.4, 61.6)
- moved PS_DC2 1.40 mm to (157.2, 65.7)
- moved C_M+1 1.37 mm to (153.9, 71.5)
Connections:
- R_SP1 pad 1: Net-(Proportional/Control1--INB) -> /V_P
- R_SP1 pad 2: /V_P -> Net-(Proportional/Control1--INB)
Routing:
- net /M+: track 19.9 -> 22.2 mm
- net /M-: track 13.7 -> 14.9 mm
Other:
- board outline added: 84 x 73.3 mm

Commit message: update
Parts:
- moved R_FP1 16.5 mm to (188.9, 84.8)
- moved R_I1 16.5 mm to (194.9, 89.5)
Other:
- board size 84 x 73.3 mm -> 50.5 x 69.8 mm
Changed lines of the file:
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@@
 	(footprint "Resistor_SMD:R_0603_1608Metric_Pad0.98x0.95mm_HandSolder"
 		(layer "F.Cu")
-		(at 175.1625 93.95)
+		(at 188.9125 84.75)
 		(descr "Resistor SMD 0603 (1608 Metric), square (rectangular) end terminal, IPC-7351 nominal with elongated pad for handsoldering. (Body size source: IPC-SM-782 page 72, https://www.pcb-3d.com/wordpress/wp-content/uploads/ipc-sm-782a_amendment_1_and_2.pdf), generated with kicad-footprint-generator")
 		(tags "resistor handsolder")
@@
 	(footprint "Resistor_SMD:R_0603_1608Metric_Pad0.98x0.95mm_HandSolder"
 		(layer "F.Cu")
-		(at 181.1625 98.7)
+		(at 194.9125 89.5)
 		(descr "Resistor SMD 0603 (1608 Metric), square (rectangular) end terminal, IPC-7351 nominal with elongated pad for handsoldering. (Body size source: IPC-SM-782 page 72, https://www.pcb-3d.com/wordpress/wp-content/uploads/ipc-sm-782a_amendment_1_and_2.pdf), generated with kicad-footprint-generator")
 		(tags "resistor handsolder")
@@
 		)
 		(property "Value" "10k"
-			(at 0 6.05 0)
+			(at 0 3.55 0)
 			(layer "F.Fab")
 			(effects
@@
 		(tags "capacitor handsolder")
 		(property "Reference" "C_BP6"
-			(at 0 -1.43 90)
+			(at 1.1 -2.65 90)
 			(layer "F.SilkS")
 			(effects
@@
 	)
 	(gr_rect
-		(start 101.5 52.2)
-		(end 185.5 125.5)
+		(start 115 54.2)
+		(end 165.5 124)
 		(stroke
 			(width 0.05)
