File: dcs_schematic_v4/dcs_schematic_v4.kicad_sch (KiCad schematic)
At the start: 71 parts, among them J1 691137710002, J2 1728307, Q1 IRLZ44N, Q2 IRLZ44N, U1 TLE2426CDR, U10 LM2917N/NOPB, U11 LM311, U2 LM311DR, U3 LM2917N/NOPB, U4 HEF4030BT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

Commit message: functional diagram, pcb layout
added kicad functional diagram schematic and started PCB design in EasyEDA
Parts:
- removed CR2: SK34A-LTP, CapstoneLibrary:SK32A-LTP_Diode, symbol Capstone_DiodeForReal:SK34A-LTP
- removed Q2: IRLZ44N, Package_TO_SOT_THT:TO-220-3_Vertical, symbol Transistor_FET:IRLZ44N
- removed U10: LM2917N/NOPB, CapstoneLibrary:LM2917M, symbol Capstone_LM2917M-NOPB:LM2917M_NOPB
- removed U11: LM311, symbol Comparator:LM311
- removed U5, U6, U7, U8: OPA2197xD, Package_SO:SOIC-8_3.9x4.9mm_P1.27mm, symbol Amplifier_Operational:OPA2197xD
- removed U9: 4077, symbol 4xxx:4077
Other:
- removed sheet Symbolic Schematic
